File: hardware/controller/controller.kicad_pcb (KiCad board)
At the start: 4 copper layers, 100 x 70 mm, 189 parts, among them J1 USB_C_Receptacle_USB2.0_14P, J10 Conn_01x01, J11 Conn_01x01, J12 Conn_02x03_Odd_Even, J2 IDC-10, J3 XT-60, J4 Conn_01x07, J5 Conn_01x01, J6 Conn_01x01, J7 Conn_01x01, J8 Conn_02x03_Odd_Even, J9 Conn_01x01, Q1 SUD50P04-08, Q10 AOD66406, Q11 AOD66406, Q12 AOD66406, Q13 AOD66406, Q2 AOD66406, Q3 AOD66406, Q4 AOD66406, Q5 AOD66406, Q6 AOD66406, Q7 AOD66406, Q8 AOD66406, Q9 AOD66406, SW1 SW_Push, SW2 SW_Push, SW3 SW_Push, SW4 SW_SPST, U1 USBLC6-2SC6, U10 LM2105D, U11 MCP6541, U12 LM2105D, U13 MCP6541, U14 LM2105D, U15 MCP6541, U16 LM2105D, U17 MCP6541, U18 LM2105D, U19 MCP6541, U2 ESP32-C3-WROOM-02, U3 STM32U535RET6, U4 nRF24L01+ 2.4Gz Mini SMD, U5 LM1117MP-3.3, U6 LV14340, U7 MPU-6050, U8 LM2105D, U9 MCP6541, Y1 8MHz

Commit message: routing
Parts:
- C19: moved to B.Cu
- moved D4 56.3 mm to (185.0, 71.2)
- moved R17 55.8 mm to (181.0, 71.2)
- moved C50 16.0 mm to (135.8, 116.2)
- moved C55 16.0 mm to (132.2, 116.2)
- moved C71 16.0 mm to (162.8, 116.2)
- moved C76 16.0 mm to (159.2, 116.2)
- moved C27 15.2 mm to (169.2, 105.8)
- moved C51 12.0 mm to (135.8, 114.2)
- moved C54 12.0 mm to (132.2, 114.2)
- moved C72 12.0 mm to (162.8, 114.2)
- moved C75 12.0 mm to (159.2, 114.2)
- moved L1 11.9 mm to (163.5, 100.0), turned to -90 degrees
- moved J2 10.2 mm to (133.2, 56.0), turned to 90 degrees
- moved C25 9.10 mm to (149.0, 93.5)
- moved C26 8.88 mm to (169.2, 100.2), turned to 90 degrees
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Routing:
- net +5V: track 0.00 -> 205.3 mm, vias 0 -> 10
- net +3.3V: track 0.00 -> 187.4 mm, vias 0 -> 38
- net GND: track 0.00 -> 130.0 mm, vias 150 -> 290
- net Net-(SW4-A): track 0.00 -> 100.2 mm, vias 0 -> 1
- net SERVO2_PWM_X: track 0.00 -> 87.4 mm, vias 0 -> 1
- net SERVO2_PWM_Y: track 0.00 -> 78.1 mm, vias 0 -> 1
- net MOTOR2_BEMF_W: track 0.00 -> 72.2 mm, vias 0 -> 2
- net MOTOR2_PWM_WL: track 0.00 -> 69.1 mm, vias 0 -> 2
- net MOTOR2_BEMF_V: track 0.00 -> 65.6 mm, vias 0 -> 2
- net MOTOR1_PWM_UH: track 0.00 -> 63.4 mm, vias 0 -> 2
- net VBUS_SENSE: track 0.00 -> 62.9 mm, vias 0 -> 3
- net MOTOR2_PWM_VL: track 0.00 -> 62.5 mm, vias 0 -> 2
- net MOTOR2_PWM_UL: track 0.00 -> 60.1 mm, vias 0 -> 2
- net SERVO1_PWM_X: track 0.00 -> 59.2 mm, vias 0 -> 1
- net MOTOR2_BEMF_U: track 0.00 -> 58.8 mm, vias 0 -> 2
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- added copper zone on F.Cu, net +5V
- added copper zone on F.Cu, net /power/BATTERY_IN
- added copper zone on F.Cu, net Net-(D3-K)
- added copper zone on F.Cu, net VBUS

Commit message: add silkscreen layer
Parts:
- added G***: LOGO, LOGO, B.Cu at (141.0, 85.0)
- added G***: LOGO, LOGO, B.Cu at (150.0, 85.0)
- added G***: LOGO, LOGO, B.Cu at (160.0, 85.5)
- moved C31 7.21 mm to (104.5, 61.5), turned to -90 degrees
- moved C32 4.47 mm to (106.5, 61.5), turned to -90 degrees
Routing:
- net GND: vias 290 -> 312
Other:
- board text added: "+"
- board text added: "-"
- board text added: "3V3"
- board text added: "5V"
- board text added: "ADC"
- board text added: "BATTERY"
- board text added: "CMP"
- board text added: "CS"
- board text added: "ESP EN ESP BOOT"
- board text added: "ESP LED"
- board text added: "G"
- board text added: "GND"
- board text added: "Hogger^2 Controller V1.0 by Eryk Możdżeń November 2024"
- board text added: "INT"
- board text added: "JLCJLCJLCJLC"
- board text added: "MISO"
- board text added: "MOSI"
- board text added: "MOTOR 1"
- board text added: "MOTOR 2"
- board text added: "NC"
- board text added: "OFF"
- board text added: "ON"
- board text added: "OPTICAL FLOW"
- board text added: "POWER"
- board text added: "PWM"
- board text added: "RST"
- board text added: "S"
- board text added: "SCK"
- board text added: "SERVO1"
- board text added: "SERVO2"
- board text added: "STM LED"
- board text added: "STM RST"
- board text added: "SWCLK"
- board text added: "SWD"
- board text added: "SWDIO"
- board text added: "SWO"
- board text added: "U"
- board text added: "USB"
- board text added: "V"
- board text added: "W"
- board text added: "X"
- board text added: "Y"
- board text added: "Z"
