File: hardware/controller/hog1.kicad_sch (KiCad schematic)
At the start: 58 parts, among them J5 Conn_01x01, J6 Conn_01x01, J7 Conn_01x01, J8 Conn_02x03_Odd_Even, Q2 AOD66406, Q3 AOD66406, Q4 AOD66406, Q5 AOD66406, Q6 AOD66406, Q7 AOD66406, U10 LM2105D, U11 LMV331, U12 LM2105D, U13 LMV331, U8 LM2105D, U9 LMV331

Commit message: first real layout, change comps to MCP6541
Parts:
- removed Q2, Q3, Q4, Q5, Q6, Q7: AOD66406, Package_TO_SOT_SMD:TO-252-2, symbol Device:Q_NMOS_DGS
- removed R22, R28, R35: 10k, Resistor_SMD:R_0603_1608Metric, symbol Device:R
- removed U11, U13, U9: LMV331, Package_TO_SOT_SMD:SOT-23-5, symbol Comparator:LMV331
- added Q2, Q3, Q4, Q5, Q6, Q7: AOD66406, Package_TO_SOT_SMD:TO-252-2, symbol Device:Q_NMOS_GDS
- added U11, U13, U9: MCP6541, Package_TO_SOT_SMD:SOT-23-5, symbol Comparator:MCP6561-OT
- C36, C41, C46: value 1u/50V -> 100n/50V
- renumbered R23 to R22, R24 to R23, R25 to R24, R26 to R25, R27 to R26, R29 to R27, R30 to R28, R31 to R29, R32 to R30, R33 to R31, R34 to R32, R36 to R33, R37 to R34
Connections:
- net +3.3V: now also U11.5 (V+), U13.5 (V+), U9.5 (V+)
- net BEMF_U: now also U9.3 (+)
- net BEMF_V: now also U11.3 (+)
- net BEMF_W: now also U13.3 (+)
- net BEMF_ZERO: now also U11.4 (-), U13.4 (-), U9.4 (-)
- net GND: now also Q3.3 (S), Q5.3 (S), Q7.3 (S), U11.2 (V-), U13.2 (V-), U9.2 (V-)
- net PHASE_U: now also Q2.3 (S), Q3.2 (D)
- net PHASE_V: now also Q4.3 (S), Q5.2 (D)
- net PHASE_W: now also Q6.3 (S), Q7.2 (D)
- net VBUS: now also Q2.2 (D), Q4.2 (D), Q6.2 (D)
- net at JP1.3 (B): now also U9.1
- net at R34.2: now also Q7.1 (G)
- net at JP2.3 (B): now also U11.1
- net at JP3.3 (B): now also U13.1
- net at R29.2: now also Q5.1 (G)
- net at R31.2: now also Q6.1 (G)
- net at R23.2: now also Q3.1 (G)
- net at R20.2: now also Q2.1 (G)
- net at R25.2: now also Q4.1 (G)
