File: hardware/controller/hog2.kicad_sch (KiCad schematic)
At the start: 58 parts, among them J10 Conn_01x01, J11 Conn_01x01, J12 Conn_02x03_Odd_Even, J9 Conn_01x01, Q10 AOD66406, Q11 AOD66406, Q12 AOD66406, Q13 AOD66406, Q8 AOD66406, Q9 AOD66406, U14 LM2105D, U15 LMV331, U16 LM2105D, U17 LMV331, U18 LM2105D, U19 LMV331

Commit message: first real layout, change comps to MCP6541
Parts:
- removed Q10, Q11, Q12, Q13, Q8, Q9: AOD66406, Package_TO_SOT_SMD:TO-252-2, symbol Device:Q_NMOS_DGS
- removed R40, R46, R53: 10k, Resistor_SMD:R_0603_1608Metric, symbol Device:R
- removed U15, U17, U19: LMV331, Package_TO_SOT_SMD:SOT-23-5, symbol Comparator:LMV331
- added Q10, Q11, Q12, Q13, Q8, Q9: AOD66406, Package_TO_SOT_SMD:TO-252-2, symbol Device:Q_NMOS_GDS
- added U15, U17, U19: MCP6541, Package_TO_SOT_SMD:SOT-23-5, symbol Comparator:MCP6561-OT
- C57, C62, C67: value 1u/50V -> 100n/50V
- renumbered R38 to R35, R39 to R36, R41 to R37, R42 to R38, R43 to R39, R44 to R40, R45 to R41, R47 to R42, R48 to R43, R49 to R44, R50 to R45, R51 to R46, R52 to R47, R54 to R48, R55 to R49
Connections:
- net +3.3V: now also U15.5 (V+), U17.5 (V+), U19.5 (V+)
- net BEMF_U: now also U15.3 (+)
- net BEMF_V: now also U17.3 (+)
- net BEMF_W: now also U19.3 (+)
- net BEMF_ZERO: now also U15.4 (-), U17.4 (-), U19.4 (-)
- net GND: now also Q11.3 (S), Q13.3 (S), Q9.3 (S), U15.2 (V-), U17.2 (V-), U19.2 (V-)
- net PHASE_U: now also Q8.3 (S), Q9.2 (D)
- net PHASE_V: now also Q10.3 (S), Q11.2 (D)
- net PHASE_W: now also Q12.3 (S), Q13.2 (D)
- net VBUS: now also Q10.2 (D), Q12.2 (D), Q8.2 (D)
- net at JP5.3 (B): now also U17.1
- net at R40.2: now also Q10.1 (G)
- net at JP6.3 (B): now also U19.1
- net at JP4.3 (B): now also U15.1
- net at R44.2: now also Q11.1 (G)
- net at R35.2: now also Q8.1 (G)
- net at R49.2: now also Q13.1 (G)
- net at R46.2: now also Q12.1 (G)
- net at R38.2: now also Q9.1 (G)
