File: hardware/controller/power.kicad_sch (KiCad schematic)
At the start: 26 parts, among them J3 XT-60, Q1 SUD50P04-08, SW4 SW_SPST, U5 LM1117MP-3.3, U6 LV14340

Commit message: full layout, edge power switch
Parts:
- SW4: footprint Button_Switch_THT:SW_CK_JS202011CQN_DPDT_Straight -> hogger2:JS102011SAQN
Changed lines of the file:
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@@
 		(dnp no)
 		(fields_autoplaced yes)
-		(property "Reference" "#PWR053"
+		(property "Reference" "#PWR054"
 			(at 195.58 115.57 0)
 			(effects
@@
 			(project "controller"
 				(path "/b81e4285-7ba7-4843-ab37-49bb8c6c135f/54c19fa3-aa0d-4e7d-a7c9-c109aa98901f"
-					(reference "#PWR053")
+					(reference "#PWR054")
 					(unit 1)
 				)
@@
 		(dnp no)
 		(fields_autoplaced yes)
-		(property "Reference" "#PWR056"
+		(property "Reference" "#PWR057"
 			(at 167.64 130.81 0)
 			(effects
@@
 			(project "controller"
 				(path "/b81e4285-7ba7-4843-ab37-49bb8c6c135f/54c19fa3-aa0d-4e7d-a7c9-c109aa98901f"
-					(reference "#PWR056")
+					(reference "#PWR057")
 					(unit 1)
 				)
@@
 		(dnp no)
 		(fields_autoplaced yes)
-		(property "Reference" "#PWR050"
+		(property "Reference" "#PWR051"
 			(at 167.64 73.66 0)
 			(effects
@@
 			(project "controller"
 				(path "/b81e4285-7ba7-4843-ab37-49bb8c6c135f/54c19fa3-aa0d-4e7d-a7c9-c109aa98901f"
-					(reference "#PWR050")
+					(reference "#PWR051")
 					(unit 1)
 				)
@@
 			)
 		)
-		(property "Footprint" "Button_Switch_THT:SW_CK_JS202011CQN_DPDT_Straight"
+		(property "Footprint" "hogger2:JS102011SAQN"
 			(at 77.47 71.12 0)
 			(effects
@@
 		(dnp no)
 		(fields_autoplaced yes)
-		(property "Reference" "#PWR049"
+		(property "Reference" "#PWR050"
 			(at 157.48 73.66 0)
 			(effects
@@
 			(project "controller"
 				(path "/b81e4285-7ba7-4843-ab37-49bb8c6c135f/54c19fa3-aa0d-4e7d-a7c9-c109aa98901f"
-					(reference "#PWR049")
+					(reference "#PWR050")
 					(unit 1)
 				)
@@
 		(dnp no)
 		(fields_autoplaced yes)
-		(property "Reference" "#PWR058"
+		(property "Reference" "#PWR059"
 			(at 76.2 138.43 0)
 			(effects
@@
 			(project "controller"
 				(path "/b81e4285-7ba7-4843-ab37-49bb8c6c135f/54c19fa3-aa0d-4e7d-a7c9-c109aa98901f"
-					(reference "#PWR058")
+					(reference "#PWR059")
 					(unit 1)
 				)
@@
 		(dnp no)
 		(fields_autoplaced yes)
-		(property "Reference" "#PWR046"
+		(property "Reference" "#PWR047"
 			(at 92.71 49.53 0)
 			(effects
@@
 			(project "controller"
 				(path "/b81e4285-7ba7-4843-ab37-49bb8c6c135f/54c19fa3-aa0d-4e7d-a7c9-c109aa98901f"
-					(reference "#PWR046")
+					(reference "#PWR047")
 					(unit 1)
 				)
@@
 		(dnp no)
 		(fields_autoplaced yes)
-		(property "Reference" "#PWR064"
+		(property "Reference" "#PWR065"
 			(at 180.34 154.94 0)
 			(effects
@@
 			(project "controller"
 				(path "/b81e4285-7ba7-4843-ab37-49bb8c6c135f/54c19fa3-aa0d-4e7d-a7c9-c109aa98901f"
-					(reference "#PWR064")
+					(reference "#PWR065")
 					(unit 1)
 				)
@@
 		(dnp no)
 		(fields_autoplaced yes)
-		(property "Reference" "#PWR060"
+		(property "Reference" "#PWR061"
 			(at 102.87 138.43 0)
 			(effects
@@
 			(project "controller"
 				(path "/b81e4285-7ba7-4843-ab37-49bb8c6c135f/54c19fa3-aa0d-4e7d-a7c9-c109aa98901f"
-					(reference "#PWR060")
+					(reference "#PWR061")
 					(unit 1)
 				)
@@
 		(dnp no)
 		(fields_autoplaced yes)
-		(property "Reference" "#PWR062"
+		(property "Reference" "#PWR063"
 			(at 30.48 154.94 0)
 			(effects
@@
 			(project "controller"
 				(path "/b81e4285-7ba7-4843-ab37-49bb8c6c135f/54c19fa3-aa0d-4e7d-a7c9-c109aa98901f"
-					(reference "#PWR062")
+					(reference "#PWR063")
 					(unit 1)
 				)
@@
 		(dnp no)
 		(fields_autoplaced yes)
-		(property "Reference" "#PWR051"
+		(property "Reference" "#PWR052"
 			(at 77.47 82.55 0)
 			(effects
@@
 			(project "controller"
 				(path "/b81e4285-7ba7-4843-ab37-49bb8c6c135f/54c19fa3-aa0d-4e7d-a7c9-c109aa98901f"
-					(reference "#PWR051")
+					(reference "#PWR052")
 					(unit 1)
 				)
@@
 		(dnp no)
 		(fields_autoplaced yes)
-		(property "Reference" "#PWR063"
+		(property "Reference" "#PWR064"
 			(at 36.83 154.94 0)
 			(effects
@@
 			(project "controller"
 				(path "/b81e4285-7ba7-4843-ab37-49bb8c6c135f/54c19fa3-aa0d-4e7d-a7c9-c109aa98901f"
-					(reference "#PWR063")
+					(reference "#PWR064")
 					(unit 1)
 				)
@@
 		(dnp no)
 		(fields_autoplaced yes)
-		(property "Reference" "#PWR065"
+		(property "Reference" "#PWR066"
 			(at 116.84 156.21 0)
 			(effects
@@
 			(project "controller"
 				(path "/b81e4285-7ba7-4843-ab37-49bb8c6c135f/54c19fa3-aa0d-4e7d-a7c9-c109aa98901f"
-					(reference "#PWR065")
+					(reference "#PWR066")
 					(unit 1)
 				)
@@
 		(dnp no)
 		(fields_autoplaced yes)
-		(property "Reference" "#PWR055"
+		(property "Reference" "#PWR056"
 			(at 116.84 125.73 0)
 			(effects
@@
 			(project "controller"
 				(path "/b81e4285-7ba7-4843-ab37-49bb8c6c135f/54c19fa3-aa0d-4e7d-a7c9-c109aa98901f"
-					(reference "#PWR055")
+					(reference "#PWR056")
 					(unit 1)
 				)
@@
 		(dnp no)
 		(fields_autoplaced yes)
-		(property "Reference" "#PWR048"
+		(property "Reference" "#PWR049"
 			(at 54.61 58.42 0)
 			(effects
@@
 			(project "controller"
 				(path "/b81e4285-7ba7-4843-ab37-49bb8c6c135f/54c19fa3-aa0d-4e7d-a7c9-c109aa98901f"
-					(reference "#PWR048")
+					(reference "#PWR049")
 					(unit 1)
 				)
@@
 		(dnp no)
 		(fields_autoplaced yes)
-		(property "Reference" "#PWR066"
+		(property "Reference" "#PWR067"
 			(at 53.34 157.48 0)
 			(effects
@@
 			(project "controller"
 				(path "/b81e4285-7ba7-4843-ab37-49bb8c6c135f/54c19fa3-aa0d-4e7d-a7c9-c109aa98901f"
-					(reference "#PWR066")
+					(reference "#PWR067")
 					(unit 1)
 				)
@@
 		(dnp no)
 		(fields_autoplaced yes)
-		(property "Reference" "#PWR047"
+		(property "Reference" "#PWR048"
 			(at 157.48 53.34 0)
 			(effects
@@
 			(project "controller"
 				(path "/b81e4285-7ba7-4843-ab37-49bb8c6c135f/54c19fa3-aa0d-4e7d-a7c9-c109aa98901f"
-					(reference "#PWR047")
+					(reference "#PWR048")
 					(unit 1)
 				)
@@
 		(dnp no)
 		(fields_autoplaced yes)
-		(property "Reference" "#PWR052"
+		(property "Reference" "#PWR053"
 			(at 139.7 115.57 0)
 			(effects
@@
 			(project "controller"
 				(path "/b81e4285-7ba7-4843-ab37-49bb8c6c135f/54c19fa3-aa0d-4e7d-a7c9-c109aa98901f"
-					(reference "#PWR052")
+					(reference "#PWR053")
 					(unit 1)
 				)
@@
 		(dnp no)
 		(fields_autoplaced yes)
-		(property "Reference" "#PWR061"
+		(property "Reference" "#PWR062"
 			(at 160.02 147.32 0)
 			(effects
@@
 			(project "controller"
 				(path "/b81e4285-7ba7-4843-ab37-49bb8c6c135f/54c19fa3-aa0d-4e7d-a7c9-c109aa98901f"
-					(reference "#PWR061")
+					(reference "#PWR062")
 					(unit 1)
 				)
@@
 		(dnp no)
 		(fields_autoplaced yes)
-		(property "Reference" "#PWR057"
+		(property "Reference" "#PWR058"
 			(at 30.48 133.35 0)
 			(effects
@@
 			(project "controller"
 				(path "/b81e4285-7ba7-4843-ab37-49bb8c6c135f/54c19fa3-aa0d-4e7d-a7c9-c109aa98901f"
-					(reference "#PWR057")
+					(reference "#PWR058")
 					(unit 1)
 				)
@@
 		(dnp no)
 		(fields_autoplaced yes)
-		(property "Reference" "#PWR054"
+		(property "Reference" "#PWR055"
 			(at 30.48 120.65 0)
 			(effects
@@
 			(project "controller"
 				(path "/b81e4285-7ba7-4843-ab37-49bb8c6c135f/54c19fa3-aa0d-4e7d-a7c9-c109aa98901f"
-					(reference "#PWR054")
+					(reference "#PWR055")
 					(unit 1)
 				)
@@
 		(dnp no)
 		(fields_autoplaced yes)
-		(property "Reference" "#PWR059"
+		(property "Reference" "#PWR060"
 			(at 86.36 138.43 0)
 			(effects
@@
 			(project "controller"
 				(path "/b81e4285-7ba7-4843-ab37-49bb8c6c135f/54c19fa3-aa0d-4e7d-a7c9-c109aa98901f"
-					(reference "#PWR059")
-					(unit 1)
-				)
+					(reference "#PWR060")
+					(unit 1)
+				)

Commit message: use diffrent P-MOSFET
Parts:
- removed Q1: SUD50P04-08, Package_TO_SOT_SMD:TO-252-2, symbol Transistor_FET:SUD50P04-08
- added Q1: AOD4189, Package_TO_SOT_SMD:TO-252-2, symbol Device:Q_PMOS_GDS
Connections:
- net BATTERY_IN: now also Q1.3 (S)
- net VBUS: now also Q1.2 (D)
- net at R10.2, R12.1: now also Q1.1 (G)
Other:
- note added: "Vds = 40V Vgs = 20V Id = 40A"
- note removed: "Vds = 40V Vgs = 20V Id = 50A"
Changed lines of the file:
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@@
 		)
 	)
-	(text "Vds = 40V\nVgs = 20V\nId = 50A"
+	(text "Vds = 40V\nVgs = 20V\nId = 40A"
 		(exclude_from_sim no)
 		(at 73.406 35.306 0)
@@
 	)
 	(symbol
+		(lib_id "Device:Q_PMOS_GDS")
+		(at 77.47 49.53 270)
+		(mirror x)
+		(unit 1)
+		(exclude_from_sim no)
+		(in_bom yes)
+		(on_board yes)
+		(dnp no)
+		(fields_autoplaced yes)
+		(property "Reference" "Q1"
+			(at 77.47 40.64 90)
+			(effects
+				(font
+					(size 1.27 1.27)
+				)
+			)
+		)
+		(property "Value" "AOD4189"
+			(at 77.47 43.18 90)
+			(effects
+				(font
+					(size 1.27 1.27)
+				)
+			)
+		)
+		(property "Footprint" "Package_TO_SOT_SMD:TO-252-2"
+			(at 80.01 44.45 0)
+			(effects
+				(font
+					(size 1.27 1.27)
+				)
+				(hide yes)
+			)
+		)
+		(property "Datasheet" "~"
+			(at 77.47 49.53 0)
+			(effects
+				(font
+					(size 1.27 1.27)
+				)
+				(hide yes)
+			)
+		)
+		(property "Description" "P-MOSFET transistor, gate/drain/source"
+			(at 77.47 49.53 0)
+			(effects
+				(font
+					(size 1.27 1.27)
+				)
+				(hide yes)
+			)
+		)
+		(pin "3"
+		)
+		(pin "2"
+		)
+		(pin "1"
+		)
+		(instances
+			(project ""
+				(path "/b81e4285-7ba7-4843-ab37-49bb8c6c135f/54c19fa3-aa0d-4e7d-a7c9-c109aa98901f"
+					(reference "Q1")
+					(unit 1)
+				)
+			)
+		)
+	)
+	(symbol
 		(lib_id "Connector_Generic:Conn_01x02")
 		(at 46.99 49.53 180)
@@
 					(unit 1)
 				)
-			)
-		)
-	)
-	(symbol
-		(lib_id "Transistor_FET:SUD50P04-08")
-		(at 77.47 49.53 270)
-		(mirror x)
-		(unit 1)
-		(exclude_from_sim no)
-		(in_bom yes)
-		(on_board yes)
-		(dnp no)
-		(fields_autoplaced yes)
-		(property "Reference" "Q1"
-			(at 77.47 40.64 90)
-			(effects
-				(font
-					(size 1.27 1.27)
-				)
-			)
-		)
-		(property "Value" "SUD50P04-08"
-			(at 77.47 43.18 90)
-			(effects
-				(font
-					(size 1.27 1.27)
-				)
-			)
-		)
-		(property "Footprint" "Package_TO_SOT_SMD:TO-252-2"
-			(at 75.565 44.577 0)
-			(effects
-				(font
-					(size 1.27 1.27)
-					(italic yes)
-				)
-				(justify left)
-				(hide yes)
-			)
-		)
-		(property "Datasheet" "https://www.vishay.com/docs/65594/sud50p04-08.pdf"
-			(at 73.66 44.45 0)
-			(effects
-				(font
-					(size 1.27 1.27)
-				)
-				(justify left)
-				(hide yes)
-			)
-		)
-		(property "Description" "-50A Id, -40V Vds, TrenchFET P-Channel Power MOSFET, 8.1mOhm Ron, 159nC Qg, -55 to 150 °C, TO-252-2"
-			(at 77.47 49.53 0)
-			(effects
-				(font
-					(size 1.27 1.27)
-				)
-				(hide yes)
-			)
-		)
-		(pin "1"
-		)
-		(pin "2"
-		)
-		(pin "3"
-		)
-		(instances
-			(project ""
-				(path "/b81e4285-7ba7-4843-ab37-49bb8c6c135f/54c19fa3-aa0d-4e7d-a7c9-c109aa98901f"
-					(reference "Q1")
-					(unit 1)
-				)

Commit message: bigger capacitors on step down
Parts:
- C26, C27: footprint Capacitor_SMD:C_1206_3216Metric -> Capacitor_SMD:C_1210_3225Metric
Changed lines of the file:
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@@
 			)
 		)
-		(property "Footprint" "Capacitor_SMD:C_1206_3216Metric"
+		(property "Footprint" "Capacitor_SMD:C_1210_3225Metric"
 			(at 85.3948 132.08 0)
 			(effects
@@
 			)
 		)
-		(property "Footprint" "Capacitor_SMD:C_1206_3216Metric"
+		(property "Footprint" "Capacitor_SMD:C_1210_3225Metric"
 			(at 101.9048 132.08 0)
 			(effects

Commit message: wip
Parts:
- R11: value 51k -> 47k
Changed lines of the file:
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@@
 	(title_block
 		(title "Hogger2 Controller")
-		(date "2025-02-18")
+		(date "2025-02-19")
 		(rev "V1.1")
 		(comment 4 "Author: Eryk Możdżeń")
@@
 			)
 		)
-		(property "Value" "51k"
+		(property "Value" "47k"
 			(at 154.94 54.6099 0)
 			(effects

Commit message: wip
Parts:
- renumbered C19 to C20, C20 to C21, C21 to C22, C22 to C23, C23 to C24, C24 to C25, C25 to C26, C26 to C27, C27 to C28, C28 to C29, SW4 to SW2, U5 to U4, U6 to U5

Commit message: wip elements
Parts:
- C21: value 100n/16V -> 100n/50V
- Q1: value AOD4189 -> DMPH4013SK3
Other:
- note removed: "Vds = 40V Vgs = 20V Id = 40A"
Changed lines of the file:
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@@
 	(title_block
 		(title "Hogger2 Controller")
-		(date "2025-02-22")
+		(date "2025-03-08")
 		(rev "V1.1")
 		(comment 4 "Author: Eryk Możdżeń")
@@
 		)
 	)
-	(text "Vds = 40V\nVgs = 20V\nId = 40A"
-		(exclude_from_sim no)
-		(at 73.406 35.306 0)
-		(effects
-			(font
-				(size 1.27 1.27)
-			)
-			(justify left)
-		)
-	)
 	(text "power input"
 		(exclude_from_sim no)
@@
 			)
 		)
-		(property "Value" "AOD4189"
+		(property "Value" "DMPH4013SK3"
 			(at 77.47 43.18 90)
 			(effects
@@
 			)
 		)
-		(property "Value" "100n/16V"
+		(property "Value" "100n/50V"
 			(at 71.12 113.03 90)
 			(effects
