File: hardware/controller/controller.kicad_sch (KiCad schematic)
At the start: 4 parts

Commit message: wip
Other:
- removed sheet hog1
- removed sheet hog2
- added sheet motor1 (motor1.kicad_sch)
- added sheet motor2 (motor2.kicad_sch)
- added sheet servos (servos.kicad_sch)
Changed lines of the file:
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@@
 	(title_block
 		(title "Hogger2 Controller")
-		(date "2025-02-18")
+		(date "2025-02-19")
 		(rev "V1.1")
 		(comment 4 "Author: Eryk Możdżeń")
@@
 	)
 	(sheet
-		(at 195.58 50.8)
+		(at 151.765 117.475)
 		(size 37.465 26.035)
 		(fields_autoplaced yes)
@@
 			(color 0 0 0 0.0000)
 		)
-		(property "Sheetname" "hog1"
-			(at 195.58 50.0884 0)
+		(property "Sheetname" "servos"
+			(at 151.765 116.7634 0)
 			(effects
 				(font
@@
 			)
 		)
-		(property "Sheetfile" "hog1.kicad_sch"
-			(at 195.58 77.4196 0)
+		(property "Sheetfile" "servos.kicad_sch"
+			(at 151.765 144.0946 0)
 			(effects
 				(font
@@
 			(project "controller"
 				(path "/b81e4285-7ba7-4843-ab37-49bb8c6c135f"
-					(page "7")
+					(page "8")
 				)
 			)
@@
 	)
 	(sheet
-		(at 63.5 50.8)
-		(size 38.1 59.69)
+		(at 151.765 50.8)
+		(size 37.465 26.035)
 		(fields_autoplaced yes)
 		(stroke
@@
 			(color 0 0 0 0.0000)
 		)
-		(property "Sheetname" "power"
-			(at 63.5 50.0884 0)
+		(property "Sheetname" "motor1"
+			(at 151.765 50.0884 0)
 			(effects
 				(font
@@
 			)
 		)
-		(property "Sheetfile" "power.kicad_sch"
-			(at 63.5 111.0746 0)
+		(property "Sheetfile" "motor1.kicad_sch"
+			(at 151.765 77.4196 0)
 			(effects
 				(font
@@
 			(project "controller"
 				(path "/b81e4285-7ba7-4843-ab37-49bb8c6c135f"
-					(page "3")
+					(page "7")
 				)
 			)
@@
 	)
 	(sheet
-		(at 151.13 50.8)
-		(size 38.1 59.69)
+		(at 64.135 50.8)
+		(size 37.465 26.035)
 		(fields_autoplaced yes)
 		(stroke
@@
 			(color 0 0 0 0.0000)
 		)
+		(property "Sheetname" "power"
+			(at 64.135 50.0884 0)
+			(effects
+				(font
+					(size 1.27 1.27)
+				)
+				(justify left bottom)
+			)
+		)
+		(property "Sheetfile" "power.kicad_sch"
+			(at 64.135 77.4196 0)
+			(effects
+				(font
+					(size 1.27 1.27)
+				)
+				(justify left top)
+			)
+		)
+		(instances
+			(project "controller"
+				(path "/b81e4285-7ba7-4843-ab37-49bb8c6c135f"
+					(page "3")
+				)
+			)
+		)
+	)
+	(sheet
+		(at 64.135 83.82)
+		(size 37.465 59.69)
+		(fields_autoplaced yes)
+		(stroke
+			(width 0.1524)
+			(type solid)
+		)
+		(fill
+			(color 0 0 0 0.0000)
+		)
 		(property "Sheetname" "sensors"
-			(at 151.13 50.0884 0)
+			(at 64.135 83.1084 0)
 			(effects
 				(font
@@
 		)
 		(property "Sheetfile" "sensors.kicad_sch"
-			(at 151.13 111.0746 0)
+			(at 64.135 144.0946 0)
 			(effects
 				(font
@@
 				(path "/b81e4285-7ba7-4843-ab37-49bb8c6c135f"
 					(page "4")
+				)
+			)
+		)
+	)
+	(sheet
+		(at 151.765 83.82)
+		(size 37.465 26.035)
+		(fields_autoplaced yes)
+		(stroke
+			(width 0.1524)
+			(type solid)
+		)
+		(fill
+			(color 0 0 0 0.0000)
+		)
+		(property "Sheetname" "motor2"
+			(at 151.765 83.1084 0)
+			(effects
+				(font
+					(size 1.27 1.27)
+				)
+				(justify left bottom)
+			)
+		)
+		(property "Sheetfile" "motor2.kicad_sch"
+			(at 151.765 110.4396 0)
+			(effects
+				(font
+					(size 1.27 1.27)
+				)
+				(justify left top)
+			)
+		)
+		(instances
+			(project "controller"
+				(path "/b81e4285-7ba7-4843-ab37-49bb8c6c135f"
+					(page "7")
 				)
 			)
@@
 	(sheet
 		(at 107.315 50.8)
-		(size 38.1 59.69)
+		(size 38.1 92.71)
 		(fields_autoplaced yes)
 		(stroke
@@
 		)
 		(property "Sheetfile" "microcontroller.kicad_sch"
-			(at 107.315 111.0746 0)
+			(at 107.315 144.0946 0)
 			(effects
 				(font
@@
 				)
 			)
-		)
-	)
-	(sheet
-		(at 195.58 84.455)
-		(size 37.465 26.035)
-		(fields_autoplaced yes)
-		(stroke
-			(width 0.1524)
-			(type solid)
-		)
-		(fill
-			(color 0 0 0 0.0000)
-		)
-		(property "Sheetname" "hog2"
-			(at 195.58 83.7434 0)
-			(effects
-				(font
-					(size 1.27 1.27)
-				)
-				(justify left bottom)
-			)
-		)
-		(property "Sheetfile" "hog2.kicad_sch"
-			(at 195.58 111.0746 0)
-			(effects
-				(font
-					(size 1.27 1.27)
-				)
-				(justify left top)
-			)
-		)
-		(instances
-			(project "controller"
-				(path "/b81e4285-7ba7-4843-ab37-49bb8c6c135f"
-					(page "7")
-				)
-			)

Commit message: wip
Connections:
- removed net GND: H1.1, H2.1, H3.1, H4.1
- no-connect marks 0 -> 4
Changed lines of the file:
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@@
 	(title_block
 		(title "Hogger2 Controller")
-		(date "2025-02-19")
+		(date "2025-02-20")
 		(rev "V1.1")
 		(comment 4 "Author: Eryk Możdżeń")
 	)
-	(junction
-		(at 146.05 179.07)
-		(diameter 0)
-		(color 0 0 0 0)
-	)
-	(junction
-		(at 146.05 173.99)
-		(diameter 0)
-		(color 0 0 0 0)
-	)
-	(junction
-		(at 146.05 168.91)
-		(diameter 0)
-		(color 0 0 0 0)
-	)
-	(wire
-		(pts
-			(xy 146.05 168.91) (xy 146.05 173.99)
-		)
-		(stroke
-			(width 0)
-			(type default)
-		)
-	)
-	(wire
-		(pts
-			(xy 146.05 163.83) (xy 146.05 168.91)
-		)
-		(stroke
-			(width 0)
-			(type default)
-		)
-	)
-	(wire
-		(pts
-			(xy 146.05 173.99) (xy 146.05 179.07)
-		)
-		(stroke
-			(width 0)
-			(type default)
-		)
-	)
-	(wire
-		(pts
-			(xy 148.59 173.99) (xy 146.05 173.99)
-		)
-		(stroke
-			(width 0)
-			(type default)
-		)
-	)
-	(wire
-		(pts
-			(xy 146.05 179.07) (xy 146.05 181.61)
-		)
-		(stroke
-			(width 0)
-			(type default)
-		)
-	)
-	(wire
-		(pts
-			(xy 148.59 163.83) (xy 146.05 163.83)
-		)
-		(stroke
-			(width 0)
-			(type default)
-		)
-	)
-	(wire
-		(pts
-			(xy 148.59 179.07) (xy 146.05 179.07)
-		)
-		(stroke
-			(width 0)
-			(type default)
-		)
-	)
-	(wire
-		(pts
-			(xy 148.59 168.91) (xy 146.05 168.91)
-		)
-		(stroke
-			(width 0)
-			(type default)
-		)
+	(no_connect
+		(at 148.59 163.83)
+	)
+	(no_connect
+		(at 148.59 179.07)
+	)
+	(no_connect
+		(at 148.59 173.99)
+	)
+	(no_connect
+		(at 148.59 168.91)
 	)
 	(symbol
@@
 					(unit 1)
 				)
-			)
-		)
-	)
-	(symbol
-		(lib_id "power:GND")
-		(at 146.05 181.61 0)
-		(unit 1)
-		(exclude_from_sim no)
-		(in_bom yes)
-		(on_board yes)
-		(dnp no)
-		(fields_autoplaced yes)
-		(property "Reference" "#PWR01"
-			(at 146.05 187.96 0)
-			(effects
-				(font
-					(size 1.27 1.27)
-				)
-				(hide yes)
-			)
-		)
-		(property "Value" "GND"
-			(at 146.05 186.69 0)
-			(effects
-				(font
-					(size 1.27 1.27)
-				)
-			)
-		)
-		(property "Footprint" ""
-			(at 146.05 181.61 0)
-			(effects
-				(font
-					(size 1.27 1.27)
-				)
-				(hide yes)
-			)
-		)
-		(property "Datasheet" ""
-			(at 146.05 181.61 0)
-			(effects
-				(font
-					(size 1.27 1.27)
-				)
-				(hide yes)
-			)
-		)
-		(property "Description" "Power symbol creates a global label with name \"GND\" , ground"
-			(at 146.05 181.61 0)
-			(effects
-				(font
-					(size 1.27 1.27)
-				)
-				(hide yes)
-			)
-		)
-		(pin "1"
-		)
-		(instances
-			(project ""
-				(path "/b81e4285-7ba7-4843-ab37-49bb8c6c135f"
-					(reference "#PWR01")
-					(unit 1)
-				)
