File: hardware/controller/motor2.kicad_sch (KiCad schematic)
At the start: 55 parts, among them J5 Conn_01x01, J6 Conn_01x01, J7 Conn_01x01, J8 Conn_02x03_Odd_Even, Q2 AOD66406, Q3 AOD66406, Q4 AOD66406, Q5 AOD66406, Q6 AOD66406, Q7 AOD66406, U10 LM2105D, U11 MCP6541, U12 LM2105D, U13 MCP6541, U8 LM2105D, U9 MCP6541

Commit message: wip
Parts:
- removed C38, C43, C48: 47u/50V, Capacitor_SMD:CP_Elec_6.3x7.7, symbol Device:C_Polarized
- removed C39, C44, C49: 1n, Capacitor_SMD:C_0603_1608Metric, symbol Device:C
- removed C42, C47, C55: 100n, Capacitor_SMD:C_0603_1608Metric, symbol Device:C
- removed C46: 100n/50V, Capacitor_SMD:C_0603_1608Metric, symbol Device:C
- removed C53, C54: 10u, Capacitor_SMD:C_0603_1608Metric, symbol Device:C
- removed J5, J6, J7: Conn_01x01, Connector_Wire:SolderWire-2.5sqmm_1x01_D2.4mm_OD4.4mm, symbol Connector_Generic:Conn_01x01
- removed J8: Conn_02x03_Odd_Even, Connector_PinHeader_2.54mm:PinHeader_2x03_P2.54mm_Horizontal, symbol Connector_Generic:Conn_02x03_Odd_Even
- removed JP2, JP3: SolderJumper_3_Open, Jumper:SolderJumper-3_P1.3mm_Open_RoundedPad1.0x1.5mm, symbol Jumper:SolderJumper_3_Open
- removed R26, R32: 47k, Resistor_SMD:R_0603_1608Metric, symbol Device:R
- removed R28, R33: 10k, Resistor_SMD:R_0603_1608Metric, symbol Device:R
- removed U10, U8: LM2105D, Package_SO:SOIC-8_3.9x4.9mm_P1.27mm, symbol Driver_FET:LM2105D
- removed U11, U13, U9: MCP6541, Package_TO_SOT_SMD:SOT-23-5, symbol Comparator:MCP6561-OT
- added C38, C43: 1n, Capacitor_SMD:C_0603_1608Metric, symbol Device:C
- added C39, C46, C53: 47u/50V, Capacitor_SMD:CP_Elec_6.3x7.7, symbol Device:C_Polarized
- added C48: 100n, Capacitor_SMD:C_0603_1608Metric, symbol Device:C
- added J10, J11, J9: Conn_01x01, Connector_Wire:SolderWire-2.5sqmm_1x01_D2.4mm_OD4.4mm, symbol Connector_Generic:Conn_01x01
- added J13: Conn_01x06, symbol Connector_Generic:Conn_01x06
- added J15: Conn_01x03, symbol Connector_Generic:Conn_01x03
- added JP4, JP5: SolderJumper_3_Open, Jumper:SolderJumper-3_P1.3mm_Open_RoundedPad1.0x1.5mm, symbol Jumper:SolderJumper_3_Open
- added R35: 220k, Resistor_SMD:R_0603_1608Metric, symbol Device:R
- added R36, R38, R39, R42, R44: 47k, Resistor_SMD:R_0603_1608Metric, symbol Device:R
- added R37, R41, R43: 68, Resistor_SMD:R_0603_1608Metric, symbol Device:R
- added R40: 10k, Resistor_SMD:R_0603_1608Metric, symbol Device:R
- added U10, U14, U8: MCP6541, Package_TO_SOT_SMD:SOT-23-5, symbol Comparator:MCP6561-OT
- added U15, U9: LM2105D, Package_SO:SOIC-8_3.9x4.9mm_P1.27mm, symbol Driver_FET:LM2105D
- C36: value 100n/50V -> 100n
- C37: value 100n -> 100n/50V
- C40: value 1u/50V -> 100n
- C41: value 100n/50V -> 1u/50V
- C45: value 1u/50V -> 100n/50V
- C50: value 100n -> 1n
- C51: value 10u -> 1u/50V
- C52: value 10u -> 100n/50V
- R20, R23, R25: value 100 -> 47k
- R21, R24: value 47k -> 68
- R29, R31: value 100 -> 220k
- R30: value 47k -> 10k
- R34: value 100 -> 68
Connections:
- net +3.3V: now also C36.2, C40.2, C48.2, U10.5 (V+), U14.5 (V+), U8.5 (V+); no longer C37.2
- net BEMF_U: now also JP1.3 (B), R20.2, R29.1, C38.1, U8.3 (+); no longer JP1.1 (A), R21.2, R24.1
- net BEMF_V: now also R27.2, R30.1, R31.1, C43.1, JP4.3 (B), U10.3 (+); no longer R27.1
- net BEMF_W: now also C50.1, JP5.3 (B), R35.1, R39.2, R40.1, U14.3 (+); no longer R30.1
- net BEMF_ZERO: now also R29.2, R31.2, R35.2, U10.4 (-), U14.4 (-), U8.4 (-); no longer R24.2, R27.2, R30.2
- net GND: now also C36.1, C41.1, C51.1, R25.2, R30.2, C38.2, C39.2, C43.2, C46.2, C48.1, C53.2, R38.2, R40.2, R44.2, U10.2 (V-), U14.2 (V-), U15.4 (GND), U8.2 (V-), U9.4 (GND); no longer C37.1, C45.1, C51.2, C52.2
- net PHASE_U: now also C37.2, R20.1, R23.2, J9.1 (Pin_1), U9.6 (SH); no longer C36.2, R21.1
- net PHASE_V: now also C45.2, R27.1, U12.6 (SH), J10.1 (Pin_1), R36.2; no longer C41.2
- net PHASE_W: now also C52.2, J11.1 (Pin_1), R39.1, R42.2, U15.6 (SH); no longer U12.6 (SH)
- net VBUS: now also C41.2, C51.2, C39.1, C46.1, C53.1, U15.1 (GVDD), U9.1 (GVDD); no longer C40.2, C45.2
- net at Q5.1 (G): now also R37.2, R38.1; no longer R29.2
- net at U12.8 (BST): now also C45.1
- net at U12.5 (GL): now also R37.1; no longer R34.1
- net at U12.7 (GH): now also R34.1; no longer R31.1
- net at Q6.1 (G): now also R41.2, R42.1; no longer R31.2
- net at Q2.1 (G): now also R21.2, R23.1; no longer R20.2
- net at Q3.1 (G): now also R24.2, R25.1; no longer R23.2
- net at Q4.1 (G): now also R34.2, R36.1; no longer R25.2
- net at Q7.1 (G): now also R43.2, R44.1; no longer R34.2
- removed net +5V: C50.1, C51.1, C52.1
- net MOTOR1_BEMF_U renamed MOTOR2_BEMF_U
- net MOTOR2_BEMF_U: now also J15.1 (Pin_1)
- net MOTOR1_PWM_WH renamed MOTOR2_PWM_VH
- net MOTOR2_PWM_VH: now also J13.3 (Pin_3)
- net MOTOR1_PWM_WL renamed MOTOR2_PWM_VL
- net MOTOR2_PWM_VL: now also J13.4 (Pin_4)
- new net: JP1.1 (A), U8.1
- new net: R21.1, U9.7 (GH)
- new net: JP5.1 (A), U14.1
- new net: JP4.1 (A), U10.1
- new net: R24.1, U9.5 (GL)
- new net: C37.1, U9.8 (BST)
- new net: R43.1, U15.5 (GL)
- new net: R41.1, U15.7 (GH)
- new net: C52.1, U15.8 (BST)
- new net MOTOR2_BEMF_V: J15.2 (Pin_2), JP4.2 (C)
- new net MOTOR2_BEMF_W: J15.3 (Pin_3), JP5.2 (C)
- new net MOTOR2_PWM_UH: J13.1 (Pin_1), U9.2 (INH)
- new net MOTOR2_PWM_UL: J13.2 (Pin_2), U9.3 (INL)
- new net MOTOR2_PWM_WH: J13.5 (Pin_5), U15.2 (INH)
- new net MOTOR2_PWM_WL: J13.6 (Pin_6), U15.3 (INL)
Other:
- note added: "MOTOR 2 BEMF signals conditioning"
- note added: "MOTOR 2 triple half-bridge"
- note removed: "ADC zero-cross detection"
- note removed: "MOTOR 1 BEMF signals conditioning"
- note removed: "MOTOR 1 triple half-bridge"
- note removed: "RC filter cut-off: 3.386 kHz"
- note removed: "SERVO 1 XY connectors"
- note removed: "comperator zero-cross detection"

Commit message: wip
Parts:
- J13: footprint (none) -> Connector_PinHeader_2.54mm:PinHeader_1x06_P2.54mm_Vertical
- J14: renamed from J15; footprint (none) -> Connector_PinHeader_2.54mm:PinHeader_1x03_P2.54mm_Vertical
- renumbered C35 to C54, C36 to C55, C37 to C56, C38 to C57, C39 to C58, C40 to C59, C41 to C60, C43 to C61, C45 to C62, C46 to C63, C48 to C64, C50 to C65, C51 to C66, C52 to C67, C53 to C68, J9 to J10, J10 to J11, J11 to J12, JP1 to JP4, JP4 to JP5, JP5 to JP6, Q4 to Q10, Q5 to Q11, Q6 to Q12, Q7 to Q13, Q2 to Q8, Q3 to Q9, R20 to R43, R21 to R44, R22 to R45, R23 to R46, R24 to R47, R25 to R48, R27 to R49, R29 to R50, R30 to R51, R31 to R52, R34 to R53, R35 to R54, R36 to R55, R37 to R56, R38 to R57, R39 to R58, R40 to R59, R41 to R60, R42 to R61, R43 to R62, R44 to R63, U8 to U14, U9 to U15, U10 to U16, U12 to U17, U14 to U18, U15 to U19

Commit message: wip - placement
Parts:
- removed J13: Conn_01x06, Connector_PinHeader_2.54mm:PinHeader_1x06_P2.54mm_Vertical, symbol Connector_Generic:Conn_01x06
- removed J14: Conn_01x03, Connector_PinHeader_2.54mm:PinHeader_1x03_P2.54mm_Vertical, symbol Connector_Generic:Conn_01x03
- added J12: Conn_01x09, Connector_PinHeader_2.54mm:PinHeader_1x09_P2.54mm_Vertical, symbol Connector_Generic:Conn_01x09
- renumbered J11 to J10, J12 to J11, J10 to J9
Connections:
- net MOTOR2_BEMF_U: now also J12.7 (Pin_7)
- net MOTOR2_BEMF_V: now also J12.8 (Pin_8)
- net MOTOR2_BEMF_W: now also J12.9 (Pin_9)
- net MOTOR2_PWM_UH: now also J12.1 (Pin_1)
- net MOTOR2_PWM_UL: now also J12.2 (Pin_2)
- net MOTOR2_PWM_VH: now also J12.3 (Pin_3)
- net MOTOR2_PWM_VL: now also J12.4 (Pin_4)
- net MOTOR2_PWM_WH: now also J12.5 (Pin_5)
- net MOTOR2_PWM_WL: now also J12.6 (Pin_6)
Changed lines of the file:
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@@
 	(title_block
 		(title "Hogger2 Controller")
-		(date "2025-02-20")
+		(date "2025-02-22")
 		(rev "V1.1")
 		(comment 4 "Author: Eryk Możdżeń")
@@
 	(global_label "MOTOR2_PWM_VH"
 		(shape input)
-		(at 158.75 166.37 180)
+		(at 160.02 172.72 180)
 		(fields_autoplaced yes)
 		(effects
@@
 		)
 		(property "Intersheetrefs" "${INTERSHEET_REFS}"
-			(at 139.6782 166.37 0)
+			(at 140.9482 172.72 0)
 			(effects
 				(font
@@
 	(global_label "MOTOR2_BEMF_V"
 		(shape input)
-		(at 158.75 181.61 180)
+		(at 160.02 185.42 180)
 		(fields_autoplaced yes)
 		(effects
@@
 		)
 		(property "Intersheetrefs" "${INTERSHEET_REFS}"
-			(at 140.2225 181.61 0)
+			(at 141.4925 185.42 0)
 			(effects
 				(font
@@
 	(global_label "MOTOR2_PWM_UL"
 		(shape input)
-		(at 158.75 163.83 180)
+		(at 160.02 170.18 180)
 		(fields_autoplaced yes)
 		(effects
@@
 		)
 		(property "Intersheetrefs" "${INTERSHEET_REFS}"
-			(at 139.7387 163.83 0)
+			(at 141.0087 170.18 0)
 			(effects
 				(font
@@
 	(global_label "MOTOR2_PWM_WL"
 		(shape input)
-		(at 158.75 173.99 180)
+		(at 160.02 180.34 180)
 		(fields_autoplaced yes)
 		(effects
@@
 		)
 		(property "Intersheetrefs" "${INTERSHEET_REFS}"
-			(at 139.6178 173.99 0)
+			(at 140.8878 180.34 0)
 			(effects
 				(font
@@
 	(global_label "MOTOR2_BEMF_U"
 		(shape input)
-		(at 158.75 179.07 180)
+		(at 160.02 182.88 180)
 		(fields_autoplaced yes)
 		(effects
@@
 		)
 		(property "Intersheetrefs" "${INTERSHEET_REFS}"
-			(at 139.9806 179.07 0)
+			(at 141.2506 182.88 0)
 			(effects
 				(font
@@
 	(global_label "MOTOR2_PWM_UH"
 		(shape input)
-		(at 158.75 161.29 180)
+		(at 160.02 167.64 180)
 		(fields_autoplaced yes)
 		(effects
@@
 		)
 		(property "Intersheetrefs" "${INTERSHEET_REFS}"
-			(at 139.4363 161.29 0)
+			(at 140.7063 167.64 0)
 			(effects
 				(font
@@
 	(global_label "MOTOR2_PWM_VL"
 		(shape input)
-		(at 158.75 168.91 180)
+		(at 160.02 175.26 180)
 		(fields_autoplaced yes)
 		(effects
@@
 		)
 		(property "Intersheetrefs" "${INTERSHEET_REFS}"
-			(at 139.9806 168.91 0)
+			(at 141.2506 175.26 0)
 			(effects
 				(font
@@
 	(global_label "MOTOR2_PWM_WH"
 		(shape input)
-		(at 158.75 171.45 180)
+		(at 160.02 177.8 180)
 		(fields_autoplaced yes)
 		(effects
@@
 		)
 		(property "Intersheetrefs" "${INTERSHEET_REFS}"
-			(at 139.3154 171.45 0)
+			(at 140.5854 177.8 0)
 			(effects
 				(font
@@
 	(global_label "MOTOR2_BEMF_W"
 		(shape input)
-		(at 158.75 184.15 180)
+		(at 160.02 187.96 180)
 		(fields_autoplaced yes)
 		(effects
@@
 		)
 		(property "Intersheetrefs" "${INTERSHEET_REFS}"
-			(at 139.8597 184.15 0)
+			(at 141.1297 187.96 0)
 			(effects
 				(font
@@
 	)
 	(symbol
-		(lib_id "Connector_Generic:Conn_01x06")
-		(at 163.83 166.37 0)
-		(unit 1)
-		(exclude_from_sim no)
-		(in_bom yes)
-		(on_board yes)
-		(dnp no)
-		(fields_autoplaced yes)
-		(property "Reference" "J13"
-			(at 166.37 167.6399 0)
-			(effects
-				(font
-					(size 1.27 1.27)
-				)
-				(justify left)
-			)
-		)
-		(property "Value" "Conn_01x06"
-			(at 166.37 168.9099 0)
-			(effects
-				(font
-					(size 1.27 1.27)
-				)
-				(justify left)
-				(hide yes)
-			)
-		)
-		(property "Footprint" "Connector_PinHeader_2.54mm:PinHeader_1x06_P2.54mm_Vertical"
-			(at 163.83 166.37 0)
-			(effects
-				(font
-					(size 1.27 1.27)
-				)
-				(hide yes)
-			)
-		)
-		(property "Datasheet" "~"
-			(at 163.83 166.37 0)
-			(effects
-				(font
-					(size 1.27 1.27)
-				)
-				(hide yes)
-			)
-		)
-		(property "Description" "Generic connector, single row, 01x06, script generated (kicad-library-utils/schlib/autogen/connector/)"
-			(at 163.83 166.37 0)
-			(effects
-				(font
-					(size 1.27 1.27)
-				)
-				(hide yes)
-			)
-		)
-		(pin "5"
-		)
-		(pin "2"
-		)
-		(pin "3"
-		)
-		(pin "4"
-		)
-		(pin "1"
-		)
-		(pin "6"
-		)
-		(instances
-			(project "controller"
-				(path "/b81e4285-7ba7-4843-ab37-49bb8c6c135f/a096c3cd-db90-4cf1-b1e9-dfd3d439d72f"
-					(reference "J13")
-					(unit 1)
-				)
-			)
-		)
-	)
-	(symbol
 		(lib_id "Device:C_Polarized")
 		(at 114.3 57.15 0)
@@
 		(dnp no)
 		(fields_autoplaced yes)
-		(property "Reference" "J10"
+		(property "Reference" "J9"
 			(at 123.19 21.5899 0)
 			(effects
@@
 			(project "controller"
 				(path "/b81e4285-7ba7-4843-ab37-49bb8c6c135f/a096c3cd-db90-4cf1-b1e9-dfd3d439d72f"
-					(reference "J10")
+					(reference "J9")
 					(unit 1)
 				)
@@
 		(dnp no)
 		(fields_autoplaced yes)
-		(property "Reference" "J11"
+		(property "Reference" "J10"
 			(at 123.19 25.3999 0)
 			(effects
@@
 			(project "controller"
 				(path "/b81e4285-7ba7-4843-ab37-49bb8c6c135f/a096c3cd-db90-4cf1-b1e9-dfd3d439d72f"
-					(reference "J11")
+					(reference "J10")
 					(unit 1)
 				)
@@
 	)
 	(symbol
+		(lib_id "Connector_Generic:Conn_01x09")
+		(at 165.1 177.8 0)
+		(unit 1)
+		(exclude_from_sim no)
+		(in_bom yes)
+		(on_board yes)
+		(dnp no)
+		(fields_autoplaced yes)
+		(property "Reference" "J12"
+			(at 167.64 177.7999 0)
+			(effects
+				(font
+					(size 1.27 1.27)
+				)
+				(justify left)
+			)
+		)
+		(property "Value" "Conn_01x09"
+			(at 167.64 179.0699 0)
+			(effects
+				(font
+					(size 1.27 1.27)
+				)
+				(justify left)
+				(hide yes)
+			)
+		)
+		(property "Footprint" "Connector_PinHeader_2.54mm:PinHeader_1x09_P2.54mm_Vertical"
+			(at 165.1 177.8 0)
+			(effects
+				(font
+					(size 1.27 1.27)
+				)
+				(hide yes)
+			)
+		)
+		(property "Datasheet" "~"
+			(at 165.1 177.8 0)
+			(effects
+				(font
+					(size 1.27 1.27)
+				)
+				(hide yes)
+			)
+		)
+		(property "Description" "Generic connector, single row, 01x09, script generated (kicad-library-utils/schlib/autogen/connector/)"
+			(at 165.1 177.8 0)
+			(effects
+				(font
+					(size 1.27 1.27)
+				)
+				(hide yes)
+			)
+		)
+		(pin "9"
+		)
+		(pin "2"
+		)
+		(pin "6"
+		)
+		(pin "5"
+		)
+		(pin "1"
+		)
+		(pin "4"
+		)
+		(pin "7"
+		)
+		(pin "8"
+		)
+		(pin "3"
+		)
+		(instances
+			(project "controller"
+				(path "/b81e4285-7ba7-4843-ab37-49bb8c6c135f/a096c3cd-db90-4cf1-b1e9-dfd3d439d72f"
+					(reference "J12")
+					(unit 1)
+				)
+			)
+		)
+	)
+	(symbol
 		(lib_id "Device:C")
 		(at 64.77 44.45 90)
@@
 		(dnp no)
 		(fields_autoplaced yes)
-		(property "Reference" "J12"
+		(property "Reference" "J11"
 			(at 123.19 29.2099 0)
 			(effects
@@
 			(project "controller"
 				(path "/b81e4285-7ba7-4843-ab37-49bb8c6c135f/a096c3cd-db90-4cf1-b1e9-dfd3d439d72f"
-					(reference "J12")
+					(reference "J11")
 					(unit 1)
 				)
@@
 					(unit 1)
 				)
-			)
-		)
-	)
-	(symbol
-		(lib_id "Connector_Generic:Conn_01x03")
-		(at 163.83 181.61 0)
-		(unit 1)
-		(exclude_from_sim no)
-		(in_bom yes)
-		(on_board yes)
-		(dnp no)
-		(fields_autoplaced yes)
-		(property "Reference" "J14"
-			(at 166.37 181.6099 0)
-			(effects
-				(font
-					(size 1.27 1.27)
-				)
-				(justify left)
-			)
-		)
-		(property "Value" "Conn_01x03"
-			(at 166.37 182.8799 0)
-			(effects
-				(font
-					(size 1.27 1.27)
-				)
-				(justify left)
-				(hide yes)
-			)
-		)
-		(property "Footprint" "Connector_PinHeader_2.54mm:PinHeader_1x03_P2.54mm_Vertical"
-			(at 163.83 181.61 0)
-			(effects
-				(font
-					(size 1.27 1.27)
-				)
-				(hide yes)
-			)
-		)
-		(property "Datasheet" "~"
-			(at 163.83 181.61 0)
-			(effects
-				(font
-					(size 1.27 1.27)
-				)
-				(hide yes)
-			)
-		)
-		(property "Description" "Generic connector, single row, 01x03, script generated (kicad-library-utils/schlib/autogen/connector/)"
-			(at 163.83 181.61 0)
-			(effects
-				(font
-					(size 1.27 1.27)
-				)
-				(hide yes)
-			)
-		)
-		(pin "3"
-		)
-		(pin "1"
-		)
-		(pin "2"
-		)
-		(instances
-			(project "controller"
-				(path "/b81e4285-7ba7-4843-ab37-49bb8c6c135f/a096c3cd-db90-4cf1-b1e9-dfd3d439d72f"
-					(reference "J14")
-					(unit 1)
-				)

Commit message: wip elements
Parts:
- Q10, Q11, Q12, Q13, Q8, Q9: value AOD66406 -> IPD90N04S4L04
Changed lines of the file:
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@@
 	(title_block
 		(title "Hogger2 Controller")
-		(date "2025-02-22")
+		(date "2025-03-08")
 		(rev "V1.1")
 		(comment 4 "Author: Eryk Możdżeń")
@@
 			)
 		)
-		(property "Value" "AOD66406"
+		(property "Value" "IPD90N04S4L04"
 			(at 100.33 48.26 0)
 			(effects
@@
 			)
 		)
-		(property "Value" "AOD66406"
+		(property "Value" "IPD90N04S4L04"
 			(at 100.33 168.91 0)
 			(effects
@@
 			)
 		)
-		(property "Value" "AOD66406"
+		(property "Value" "IPD90N04S4L04"
 			(at 100.33 152.4 0)
 			(effects
@@
 			)
 		)
-		(property "Value" "AOD66406"
+		(property "Value" "IPD90N04S4L04"
 			(at 100.33 64.77 0)
 			(effects
@@
 			)
 		)
-		(property "Value" "AOD66406"
+		(property "Value" "IPD90N04S4L04"
 			(at 100.33 116.84 0)
 			(effects
@@
 			)
 		)
-		(property "Value" "AOD66406"
+		(property "Value" "IPD90N04S4L04"
 			(at 100.33 100.33 0)
 			(effects

Commit message: wip routing power stages
Connections:
- net MOTOR2_BEMF_U: now also J12.1 (Pin_1); no longer J12.7 (Pin_7)
- net MOTOR2_BEMF_V: now also J12.4 (Pin_4); no longer J12.8 (Pin_8)
- net MOTOR2_BEMF_W: now also J12.7 (Pin_7); no longer J12.9 (Pin_9)
- net MOTOR2_PWM_UH: now also J12.2 (Pin_2); no longer J12.1 (Pin_1)
- net MOTOR2_PWM_UL: now also J12.3 (Pin_3); no longer J12.2 (Pin_2)
- net MOTOR2_PWM_VH: now also J12.5 (Pin_5); no longer J12.3 (Pin_3)
- net MOTOR2_PWM_VL: now also J12.6 (Pin_6); no longer J12.4 (Pin_4)
- net MOTOR2_PWM_WH: now also J12.8 (Pin_8); no longer J12.5 (Pin_5)
- net MOTOR2_PWM_WL: now also J12.9 (Pin_9); no longer J12.6 (Pin_6)
