File: hardware/controller/servos.kicad_sch (KiCad schematic)
At the start: 12 parts, among them J16 MOLEX SPOX, J5 MOLEX SPOX, U16 TXS0101DBV, U3 TXS0101DBV

Commit message: wip
Parts:
- removed C59, C62: 10u, symbol Device:C
- added C71, C75: 47u/50V, Capacitor_SMD:CP_Elec_6.3x7.7, symbol Device:C_Polarized
- C69: renamed from C56; footprint (none) -> Capacitor_SMD:C_0603_1608Metric
- C70: renamed from C57; footprint (none) -> Capacitor_SMD:C_0603_1608Metric
- C72: renamed from C58; footprint (none) -> Capacitor_SMD:C_0603_1608Metric
- C73: renamed from C60; footprint (none) -> Capacitor_SMD:C_0603_1608Metric
- C74: renamed from C61; footprint (none) -> Capacitor_SMD:C_0603_1608Metric
- C76: renamed from C63; footprint (none) -> Capacitor_SMD:C_0603_1608Metric
- J15: renamed from J5; value MOLEX SPOX -> Mini-SPOX; footprint (none) -> hogger2:Molex-MiniSPOX-22057035-5268
- J16: value MOLEX SPOX -> Mini-SPOX; footprint (none) -> hogger2:Molex-MiniSPOX-22057035-5268
- renumbered U3 to U20, U16 to U21
Connections:
- net GND: now also C71.2, C75.2
- net VBUS: now also C71.1, C75.1
- net SERVO1_TTL: now reaches J15.3 (Pin_3), U20.4 (B)
- net SERVO2_TTL: now reaches J16.3 (Pin_3), U21.4 (B)
Other:
- note added: "SERVO 1 Dynamixel TTL Multi-Drop Bus"
- note added: "SERVO 2 Dynamixel TTL Multi-Drop Bus"
- note removed: "SERVO 1 Multi-Drop Bus"
- note removed: "SERVO 2 Multi-Drop Bus"

Commit message: wip - placement
Parts:
- renumbered J15 to J13, J16 to J14
Changed lines of the file:
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@@
 	(title_block
 		(title "Hogger2 Controller")
-		(date "2025-02-20")
+		(date "2025-02-22")
 		(rev "V1.1")
 		(comment 4 "Author: Eryk Możdżeń")
@@
 		(dnp no)
 		(fields_autoplaced yes)
-		(property "Reference" "J15"
+		(property "Reference" "J13"
 			(at 160.02 53.34 0)
 			(effects
@@
 			(project ""
 				(path "/b81e4285-7ba7-4843-ab37-49bb8c6c135f/3ac54464-9759-4092-adde-e5df53f5c8cc"
-					(reference "J15")
+					(reference "J13")
 					(unit 1)
 				)
@@
 		(dnp no)
 		(fields_autoplaced yes)
-		(property "Reference" "J16"
+		(property "Reference" "J14"
 			(at 160.02 118.11 0)
 			(effects
@@
 			(project "controller"
 				(path "/b81e4285-7ba7-4843-ab37-49bb8c6c135f/3ac54464-9759-4092-adde-e5df53f5c8cc"
-					(reference "J16")
+					(reference "J14")
 					(unit 1)
 				)
